File: hardware/pcb/main-board/audio.kicad_sch (KiCad schematic)
At the start: 13 parts, among them J1002 AudioJack3, U1001 NC7WZ16P6X

Commit message: make a start on RP2040 to replace the KB pico
Other:
- title: Z88R - Z88 Recreated -> Z88R - Z88 Recreation
Changed lines of the file:
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@@
 	(paper "A4")
 	(title_block
-		(title "Z88R - Z88 Recreated")
-		(date "2025-12-19")
-		(rev "20251219WIP")
+		(title "Z88R - Z88 Recreation")
+		(date "2025-12-30")
+		(rev "20251230WIP")
 		(company "Fountain and Menadue")
 	)
