File: hardware/pcb/main-board/cm4_highspeed.kicad_sch (KiCad schematic)
At the start: 29 parts, among them J301 MIPI x40 FPC Top Contact, J302 USB_B_Micro, J303 USB_B_Micro, J304 USB_B_Micro, J305 HDMI Conn, U301 AP22653W6, U302 FE1.1s, U303 RT9742SNGV, Y301 ABLS-12.000MHZ-B4-T

Commit message: make a start on RP2040 to replace the KB pico
Other:
- title: Z88R - Z88 Recreated -> Z88R - Z88 Recreation
Changed lines of the file:
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@@
 	(paper "A4")
 	(title_block
-		(title "Z88R - Z88 Recreated")
-		(date "2025-12-19")
-		(rev "20251219WIP")
+		(title "Z88R - Z88 Recreation")
+		(date "2025-12-30")
+		(rev "20251230WIP")
 		(company "Fountain and Menadue")
 	)
