File: hardware/pcb/application-board/app_board.kicad_sch (KiCad schematic)
At the start: 43 parts, among them J101 Conn_01x04_Socket, J102 Conn_02x08_Top_Bottom, J103 Conn_01x04_Socket

Commit message: more layout work
Connections:
- net PICO_PWR: now reaches A101.39 (VSYS), A102.39 (VSYS), D101.1 (K)
Changed lines of the file:
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@@
+		)
+	)
+	(label "PICO_PWR"
+		(at 106.68 33.02 0)
+		(effects
+			(font
+				(size 1.27 1.27)
+			)
+			(justify left bottom)
 		)
 	)
