File: hardware/pcb/application-board/z88r_connection.kicad_sch (KiCad schematic)
At the start: 37 parts, among them J201 DISP_PCB x40 FPC, Q201 DMG2302U, Q202 DMG2301L

Commit message: start layout of application board
Parts:
- added C201: 100nF, Capacitor_SMD:C_0805_2012Metric_Pad1.18x1.45mm_HandSolder, symbol Device:C_Small
- added H203: PWR_555, Connector_Pin:Pin_D0.7mm_L6.5mm_W1.8mm_FlatFork, symbol Mechanical:MountingHole_Pad
- added H204: TR, Connector_Pin:Pin_D0.7mm_L6.5mm_W1.8mm_FlatFork, symbol Mechanical:MountingHole_Pad
- added H205: CV, Connector_Pin:Pin_D0.7mm_L6.5mm_W1.8mm_FlatFork, symbol Mechanical:MountingHole_Pad
- added H206: R, Connector_Pin:Pin_D0.7mm_L6.5mm_W1.8mm_FlatFork, symbol Mechanical:MountingHole_Pad
- added H207: Q, Connector_Pin:Pin_D0.7mm_L6.5mm_W1.8mm_FlatFork, symbol Mechanical:MountingHole_Pad
- added H208: DIS, Connector_Pin:Pin_D0.7mm_L6.5mm_W1.8mm_FlatFork, symbol Mechanical:MountingHole_Pad
- added H209: THR, Connector_Pin:Pin_D0.7mm_L6.5mm_W1.8mm_FlatFork, symbol Mechanical:MountingHole_Pad
- added U201: Unused 555, Package_SO:SOIC-8_3.9x4.9mm_P1.27mm, symbol Timer:LMC555xM
Connections:
- net +5V: now also J201.1 (Pin_1), J201.2 (Pin_2), J201.3 (Pin_3); no longer J201.38 (Pin_38), J201.39 (Pin_39), J201.40 (Pin_40)
- net ENABLE_APP_BOARD: now also J201.39 (Pin_39); no longer J201.2 (Pin_2)
- net GND: now also J201.15 (Pin_15), J201.25 (Pin_25), J201.30 (Pin_30), J201.33 (Pin_33), J201.40 (Pin_40), C201.2, U201.1 (GND); no longer J201.1 (Pin_1), J201.11 (Pin_11), J201.16 (Pin_16), J201.26 (Pin_26), J201.8 (Pin_8)
- net at JP204.1 (A): now also J201.8 (Pin_8); no longer J201.33 (Pin_33)
- net at JP206.1 (A): now also J201.10 (Pin_10); no longer J201.31 (Pin_31)
- net at JP227.1 (A): now also J201.35 (Pin_35); no longer J201.6 (Pin_6)
- net at JP222.1 (A): now also J201.28 (Pin_28); no longer J201.13 (Pin_13)
- net at JP226.1 (A): now also J201.34 (Pin_34); no longer J201.7 (Pin_7)
- net at JP209.1 (A): now also J201.13 (Pin_13); no longer J201.28 (Pin_28)
- net at JP224.1 (A): now also J201.31 (Pin_31); no longer J201.10 (Pin_10)
- net at JP228.1 (A): now also J201.36 (Pin_36); no longer J201.5 (Pin_5)
- net at JP201.1 (A): now also J201.5 (Pin_5); no longer J201.36 (Pin_36)
- net at JP210.1 (A): now also J201.14 (Pin_14); no longer J201.27 (Pin_27)
- net at JP212.1 (A): now also J201.17 (Pin_17); no longer J201.24 (Pin_24)
- net at JP225.1 (A): now also J201.32 (Pin_32); no longer J201.9 (Pin_9)
- net at JP213.1 (A): now also J201.18 (Pin_18); no longer J201.23 (Pin_23)
- net at JP219.1 (A): now also J201.24 (Pin_24); no longer J201.17 (Pin_17)
- net at JP216.1 (A): now also J201.21 (Pin_21); no longer J201.20 (Pin_20)
- net at JP211.1 (A): now also J201.16 (Pin_16); no longer J201.25 (Pin_25)
- net at JP205.1 (A): now also J201.9 (Pin_9); no longer J201.32 (Pin_32)
- net at J201.12 (Pin_12): now also JP208.1 (A); no longer JP223.1 (A)
- net at JP221.1 (A): now also J201.27 (Pin_27); no longer J201.14 (Pin_14)
- net at JP220.1 (A): now also J201.26 (Pin_26); no longer J201.15 (Pin_15)
- net at JP218.1 (A): now also J201.23 (Pin_23); no longer J201.18 (Pin_18)
- net at J201.19 (Pin_19): now also JP214.1 (A); no longer JP217.1 (A)
- net at JP215.1 (A): now also J201.20 (Pin_20); no longer J201.21 (Pin_21)
- net at J201.22 (Pin_22): now also JP217.1 (A); no longer JP214.1 (A)
- net at J201.29 (Pin_29): now also JP223.1 (A); no longer JP208.1 (A)
- net at JP229.1 (A): now also J201.38 (Pin_38); no longer J201.3 (Pin_3)
- net at JP207.1 (A): now also J201.11 (Pin_11); no longer J201.30 (Pin_30)
- net at JP203.1 (A): now also J201.7 (Pin_7); no longer J201.34 (Pin_34)
- net at JP202.1 (A): now also J201.6 (Pin_6); no longer J201.35 (Pin_35)
- new net: H207.1, U201.3 (Q)
- new net: H204.1, U201.2 (TR)
- new net: H206.1, U201.4 (R)
- new net: H205.1, U201.5 (CV)
- new net: H209.1, U201.6 (THR)
- new net: H208.1, U201.7 (DIS)
- new net: C201.1, H203.1, U201.8 (VCC)
Other:
- note added: "Power deliberately disconnected, it'll need either 3V3 or 5V, depending on how we use it. Ignore ERC errors here."
- moved on the sheet: J201, JP201, JP202, JP203, JP204, JP205, JP206, JP207, JP208, JP209, JP210, JP211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

Commit message: more layout work
Connections:
- net PCHAN_GATE: now reaches Q201.3 (D), Q202.1 (G), R201.2
Changed lines of the file:
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@@
+		)
+	)
+	(label "PCHAN_GATE"
+		(at 213.36 74.93 0)
+		(effects
+			(font
+				(size 1.27 1.27)
+			)
+			(justify left bottom)
 		)
 	)
